Commit message: changed name of wheels

File: description/ros2_control.xacro (robot description, xacro)
@@ -14,5 +14,5 @@
             <state_interface name="velocity" />
         <joint>
-        <joint name="back_left_wheel_joint">
+        <joint name="rear_left_wheel_joint">
             <command_interface name = velocity>
                 <param name="min">-10</param>
@@ -30,5 +30,5 @@
             <state_interface name="velocity" />
         <joint>
-        <joint name="back_right_wheel_joint">
+        <joint name="rear_right_wheel_joint">
             <command_interface name = velocity>
                 <param name="min">-10</param>
